File: PCBs/pressurePlate/pressurePlate.kicad_pcb (KiCad board)
At the start: 2 copper layers, 145.5 x 146.3 mm, 21 parts, among them IC1 MCP23017ML

Commit message: AHHHHHHHHH
Parts:
- removed C3: 10uF, 0805-NO
- added Cap1: CP_Radial_D4.0mm_P2.00mm, Capacitor_THT:CP_Radial_D4.0mm_P2.00mm, F.Cu at (35.1, 173.2)
- added D1: GREEN, CHIPLED_0603_NOOUTLINE, F.Cu at (104.4, 166.5)
- added FID3: FIDUCIAL_1MM, FIDUCIAL_1MM, F.Cu at (105.6, 173.6)
- added GND: SolderWirePad_1x01_SMD_1x2mm, Connector_Wire:SolderWirePad_1x01_SMD_1x2mm, F.Cu at (25.9, 166.1)
- added GPIO: PinHeader_1x05_P2.54mm_Vertical, Connector_PinHeader_2.54mm:PinHeader_1x05_P2.54mm_Vertical, F.Cu at (44.2, 175.3)
- added R2: 10k, 0603-NO, F.Cu at (106.7, 166.9)
- added SJ1: , SOLDERJUMPER_CLOSEDWIRE, B.Cu at (105.3, 167.3)
- added VCC: SolderWirePad_1x01_SMD_1x2mm, Connector_Wire:SolderWirePad_1x01_SMD_1x2mm, F.Cu at (26.7, 23.4)
- moved JP7 19.4 mm to (128.4, 166.5)
- moved JP2 19.4 mm to (128.4, 176.7)
- moved JP6 19.4 mm to (128.4, 164.0)
- moved JP8 19.4 mm to (128.4, 174.1)
- moved R3 19.4 mm to (108.4, 170.9)
- moved ADDR0 19.4 mm to (111.5, 167.1)
- moved ADDR1 19.4 mm to (114.3, 167.1)
- moved ADDR2 19.4 mm to (117.2, 167.1)
- moved C1 19.4 mm to (113.4, 166.2)
- moved C2 19.4 mm to (108.2, 173.7)
- moved IC1 19.4 mm to (115.2, 170.7)
- moved JP1 19.4 mm to (111.9, 164.0)
- moved JP5 19.4 mm to (111.9, 176.7)
- moved R1 19.4 mm to (109.4, 167.4)
Routing:
- net (no net): track 5186.3 -> 8780.7 mm, vias 95 -> 193
Other:
- board size 145.5 x 146.3 mm -> 145.5 x 158.5 mm
- board text added: "16 IO Expander"
- board text added: "GND VCC SIG SDA SCL"

Commit message: ahhhhhhh
Routing:
- net (no net): track 8780.7 -> 8789.5 mm, vias 193 -> 195
Changed lines of the file:
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@@
   (segment (start 43.18 100.076) (end 54.356 100.076) (width 0.25) (layer "F.Cu") (net 0))
   (segment (start 57.404 97.028) (end 57.404 92.456) (width 0.25) (layer "F.Cu") (net 0))
+  (segment (start 99.187 65.151) (end 99.568 65.532) (width 0.25) (layer "F.Cu") (net 0))
   (segment (start 131.7521 171.338) (end 133.5151 173.101) (width 0.254) (layer "F.Cu") (net 0))
   (segment (start 162.052 61.468) (end 162.052 160.274) (width 0.25) (layer "F.Cu") (net 0))
@@
   (segment (start 153.67 71.882) (end 153.67 73.66) (width 0.25) (layer "F.Cu") (net 0))
   (segment (start 109.728 151.892) (end 109.728 152.4) (width 0.25) (layer "F.Cu") (net 0))
+  (segment (start 99.568 65.532) (end 99.568 67.056) (width 0.25) (layer "F.Cu") (net 0))
   (segment (start 31.496 26.162) (end 31.496 26.67) (width 0.25) (layer "F.Cu") (net 0))
   (segment (start 162.052 160.274) (end 163.068 161.29) (width 0.25) (layer "F.Cu") (net 0))
@@
   (segment (start 115.022687 165.227) (end 115.7605 164.489188) (width 0.3048) (layer "F.Cu") (net 0))
   (segment (start 75.438 80.518) (end 74.168 81.788) (width 0.25) (layer "F.Cu") (net 0))
+  (segment (start 100.457 63.881) (end 100.965 63.881) (width 0.25) (layer "F.Cu") (net 0))
   (segment (start 42.672 153.035) (end 43.18 153.543) (width 0.25) (layer "F.Cu") (net 0))
   (segment (start 149.352 112.903) (end 148.082 114.173) (width 0.25) (layer "F.Cu") (net 0))
@@
   (segment (start 128.4605 173.379032) (end 128.4605 174.6504) (width 0.254) (layer "F.Cu") (net 0))
   (segment (start 77.216 25.908) (end 77.216 34.798) (width 0.25) (layer "F.Cu") (net 0))
+  (segment (start 100.965 63.881) (end 101.092 64.008) (width 0.25) (layer "F.Cu") (net 0))
   (segment (start 129.032 155.448) (end 120.396 155.448) (width 0.25) (layer "F.Cu") (net 0))
   (segment (start 31.75 41.656) (end 33.274 41.656) (width 0.25) (layer "F.Cu") (net 0))
@@
   (segment (start 105.664 115.824) (end 105.664 113.792) (width 0.25) (layer "F.Cu") (net 0))
   (segment (start 132.588 117.602) (end 132.588 116.84) (width 0.25) (layer "F.Cu") (net 0))
+  (segment (start 100.457 63.881) (end 96.852 63.881) (width 0.25) (layer "F.Cu") (net 0))
   (segment (start 100.076 122.936) (end 100.076 142.24) (width 0.25) (layer "F.Cu") (net 0))
   (segment (start 112.1156 173.0495) (end 112.1156 173.5455) (width 0.254) (layer "F.Cu") (net 0))
@@
   (segment (start 104.8051 169.807) (end 104.3178 170.2943) (width 0.3048) (layer "F.Cu") (net 0))
   (segment (start 82.296 41.402) (end 77.47 41.402) (width 0.25) (layer "F.Cu") (net 0))
+  (segment (start 96.852 65.151) (end 99.187 65.151) (width 0.25) (layer "F.Cu") (net 0))
   (segment (start 71.628 156.464) (end 71.628 160.02) (width 0.25) (layer "F.Cu") (net 0))
   (segment (start 110.6343 169.388) (end 110.5281 169.4942) (width 0.254) (layer "F.Cu") (net 0))
@@
   (segment (start 104.648 112.776) (end 109.728 107.696) (width 0.25) (layer "F.Cu") (net 0))
   (segment (start 130.81 40.64) (end 135.128 40.64) (width 0.25) (layer "F.Cu") (net 0))
+  (segment (start 100.584 64.008) (end 100.457 63.881) (width 0.25) (layer "F.Cu") (net 0))
   (segment (start 112.5271 168.738) (end 112.5271 168.369) (width 0.254) (layer "F.Cu") (net 0))
   (segment (start 140.462 117.094) (end 135.763 121.793) (width 0.25) (layer "F.Cu") (net 0))
@@
   (via (at 159.004 70.612) (size 0.8) (drill 0.4) (layers "F.Cu" "B.Cu") (net 0))
   (via (at 92.71 41.402) (size 0.8) (drill 0.4) (layers "F.Cu" "B.Cu") (net 0))
+  (via (at 101.092 64.008) (size 0.8) (drill 0.4) (layers "F.Cu" "B.Cu") (net 0))
   (via (at 47.244 152.4) (size 0.8) (drill 0.4) (layers "F.Cu" "B.Cu") (net 0))
   (via (at 123.19 132.842) (size 0.8) (drill 0.4) (layers "F.Cu" "B.Cu") (net 0))
@@
   (via (at 160.528 70.612) (size 0.8) (drill 0.4) (layers "F.Cu" "B.Cu") (net 0))
   (via (at 107.696 56.642) (size 0.8) (drill 0.4) (layers "F.Cu" "B.Cu") (net 0))
+  (via (at 99.568 67.056) (size 0.8) (drill 0.4) (layers "F.Cu" "B.Cu") (net 0))
   (via (at 146.304 156.464) (size 0.8) (drill 0.4) (layers "F.Cu" "B.Cu") (net 0))
   (via (at 115.316 48.768) (size 0.8) (drill 0.4) (layers "F.Cu" "B.Cu") (net 0))
